File: macropad/macropad.kicad_sch (KiCad schematic)
At the start: 14 parts, among them SW1 SW_Push, U1 ATmega32U4-A, Y1 16 MHz

Commit message: finished schematic
Parts:
- added D1, D2, D3, D4: D_Small, Diode_SMD:D_SOD-123, symbol Device:D_Small
- added F1: Polyfuse_Small, Fuse:Fuse_1206_3216Metric, symbol Device:Polyfuse_Small
- added MX1, MX2, MX3, MX4: MX-NoLED, MX_Only:MXOnly-1U-NoLED, symbol MX_Alps_Hybrid:MX-NoLED
- added USB1: Molex-0548190589, random-keyboard-parts:Molex-0548190589, symbol random-keyboard-parts:Molex-0548190589
- C1, C2, C3, C4, C5, C6, C7: footprint (none) -> Capacitor_SMD:C_0805_2012Metric
- R1, R2, R3, R4: footprint (none) -> Resistor_SMD:R_0805_2012Metric
- SW1: footprint (none) -> random-keyboard-parts:SKQG-1155865
- Y1: footprint (none) -> Package_QFP:TQFP-44_10x10mm_P0.8mm
Connections:
- net +5V: now also F1.2
- net GND: now also USB1.1 (GND)
- net D+: now reaches R2.1
- net D+: now also USB1.3 (D+)
- net D-: now reaches R3.1
- net D-: now also USB1.4 (D-)
- net ROW0: now reaches U1.27 (PD7)
- net ROW0: now also D1.1 (K), D2.1 (K)
- net COL1: now reaches U1.28 (PB4)
- net COL1: now also MX2.1 (COL), MX3.1 (COL)
- net COL0: now reaches U1.29 (PB5)
- net COL0: now also MX1.1 (COL), MX4.1 (COL)
- net ROW1: now reaches U1.30 (PB6)
- net ROW1: now also D3.1 (K), D4.1 (K)
- new net: D1.2 (A), MX1.2 (ROW)
- new net: D2.2 (A), MX2.2 (ROW)
- new net: D3.2 (A), MX3.2 (ROW)
- new net: D4.2 (A), MX4.2 (ROW)
- new net VCC: F1.1, USB1.5 (VBUS)
Other:
- moved on the sheet: R1

Commit message: pcb layout
Parts:
- Y1: footprint Package_QFP:TQFP-44_10x10mm_P0.8mm -> Crystal:Crystal_SMD_3225-4Pin_3.2x2.5mm
Connections:
- no-connect marks 0 -> 2
Changed lines of the file:
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@@
 		(color 0 0 0 0)
+	)
+	(no_connect
+		(at 50.8 27.94)
+	)
+	(no_connect
+		(at 50.8 38.1)
 	)
 	(wire
@@
 			)
 		)
-		(property "Footprint" "Package_QFP:TQFP-44_10x10mm_P0.8mm"
+		(property "Footprint" "Crystal:Crystal_SMD_3225-4Pin_3.2x2.5mm"
 			(at 78.74 60.96 0)
 			(effects
